File: redox/pcb/rev1.0lp/kicad_files/redox_rev1.kicad_pcb (KiCad board)
At the start: 2 copper layers, 162.2 x 126.5 mm, 86 parts, among them K0 KEYSW, K1 KEYSW, K10 KEYSW, K11 KEYSW, K12 KEYSW, K13 KEYSW, K14 KEYSW, K15 KEYSW, K16 KEYSW, K2 KEYSW, K20 KEYSW, K21 KEYSW, K22 KEYSW, K23 KEYSW, K24 KEYSW, K25 KEYSW, K26 KEYSW, K3 KEYSW, K30 KEYSW, K31 KEYSW, K32 KEYSW, K33 KEYSW, K34 KEYSW, K35 KEYSW, K36 KEYSW, K4 KEYSW, K40 KEYSW, K41 KEYSW, K42 KEYSW, K43 KEYSW, K44 KEYSW, K45 KEYSW, K46 KEYSW, K5 KEYSW, K6 KEYSW, U1 ProMicro

Commit message: move switch footprints into local folder and change schematic to use them instead
Parts:
- K0, K10, K20, K30, K44: footprint PCM_Switch_Keyboard_Hotswap_Kailh:SW_Hotswap_Kailh_Choc_V1V2_1.25u -> redox_footprints:SW_Hotswap_Kailh_Choc_V1V2_1.25u
- K1, K11, K12, K13, K14, K15, K2, K21, K22, K23, K24, K25, K26, K3, K31, K32, K33, K34, K35, K36, K4, K40, K41, K42, K43, K5, K6: footprint PCM_Switch_Keyboard_Hotswap_Kailh:SW_Hotswap_Kailh_Choc_V1V2_1.00u -> redox_footprints:SW_Hotswap_Kailh_Choc_V1V2_1.00u
- K16, K45, K46: footprint PCM_Switch_Keyboard_Hotswap_Kailh:SW_Hotswap_Kailh_Choc_V1V2_1.50u -> redox_footprints:SW_Hotswap_Kailh_Choc_V1V2_1.50u
Routing:
- net /Net-(D45-Pad2): track 6.51 -> 0.00 mm
- net (no net): track 0.00 -> 6.51 mm
